File: Teensy35Mega.sch (KiCad schematic (older format))
At the start: 28 parts, among them CON1 BARREL_JACK, J1 CONN_01X03, J2 CONN_01X02, P1 CONN_01X08, P10 CONN_02X18, P11 CONN_01X24, P12 CONN_01X08, P13 CONN_01X08, P14 CONN_01X08, P15 CONN_02X03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

Commit message: Updated P8 connections & Layout
Updated P8 connections. per @boelle on PRJC Forum
Connections:
- net at P10.28 (P28): now also P8.7 (P7); no longer P8.8 (P8)
- net at P10.30 (P30): now also P8.5 (P5); no longer P8.6 (P6)
- net at P10.32 (P32): now also P8.3 (P3); no longer P8.4 (P4)
- net at P10.34 (P34): now also P8.1 (P1); no longer P8.2 (P2)
Changed lines of the file:
@@
 F 3 "" H 4250 5700 50  0000 C CNN
 	1    4250 6900
-	-1   0    0    1
+	1    0    0    1
 $EndComp
 $Comp
